Commit message: simplified vehicle model

File: a2d2_ros_preparer/urdf/audi_a2d2.urdf (robot description, URDF)
Before this commit: robot audi_a2d2, 2 links, 1 joints
Links:
- removed link upper_link
- link base_link: geometry visual box size=3.2 2.5 0.6; visual box size=5.0 2.5 0.9
Joints:
- removed joint base_to_upper
